File: pcb/Eastern Style Keyboard/Eastern Style Keyboard.kicad_pcb (KiCad board)
At the start: 2 copper layers, 4 x 3.7 mm, 255 parts, among them SW1 RotaryEncoder_Switch, SW10 SW_Push, SW11 SW_Push, SW12 SW_Push, SW13 SW_Push, SW14 SW_Push, SW15 SW_Push, SW16 SW_Push, SW17 SW_Push, SW18 SW_Push, SW19 SW_Push, SW2 SW_Push, SW20 SW_Push, SW21 SW_Push, SW22 SW_Push, SW23 SW_Push, SW24 SW_Push, SW25 SW_Push, SW26 SW_Push, SW27 SW_Push, SW28 SW_Push, SW29 SW_Push, SW3 SW_Push, SW30 SW_Push, SW31 SW_Push, SW32 SW_Push, SW33 SW_Push, SW34 SW_Push, SW35 SW_Push, SW36 SW_Push, SW37 SW_Push, SW38 SW_Push, SW39 SW_Push, SW4 SW_Push, SW40 SW_Push, SW41 SW_Push, SW42 SW_Push, SW43 SW_Push, SW44 SW_Push, SW45 SW_Push, SW46 SW_Push, SW47 SW_Push, SW48 SW_Push, SW49 SW_Push, SW5 SW_Push, SW50 SW_Push, SW51 SW_Push, SW52 SW_Push, SW53 SW_Push, SW54 SW_Push, SW55 SW_Push, SW56 SW_Push, SW57 SW_Push, SW58 SW_Push, SW59 SW_Push, SW6 SW_Push, SW60 SW_Push, SW61 SW_Push, SW62 SW_Push, SW63 SW_Push, SW64 SW_Push, SW65 SW_Push, SW66 SW_Push, SW67 SW_Push, SW68 SW_Push, SW69 SW_Push, SW7 SW_Push, SW70 SW_Push, SW71 SW_Push, SW72 SW_Push, SW73 SW_Push, SW74 SW_Push, SW75 SW_Push, SW76 SW_Push, SW8 SW_Push, SW9 SW_Push, U1 ER_OLEDM0.91_1x-I2C

Commit message: Fix 2 of 6 electrical shorts flagged by PCB DRC on Eastern Style Keyboard
The board's DRC.rpt on disk was stale (board saved 62 min after the report
ran) and no longer reflects the current layout. A fresh DRC pass found 149
active violations, including 6 real shorting_items errors.

Diagnosed root cause for 2 of them: the MX stabilizer footprints (S3, S4)
have unplated/plated mounting holes with no net assigned, and the Row 2 /
Row 3 matrix traces were routed directly across those holes, shorting the
row net to the stabilizer's bare copper. Rerouted both traces around the
hole keepout (>=2.3mm clearance) instead of through it.

Also deleted a small orphaned, netless B.Cu trace stub near S3 that was
the source of 2 track_dangling warnings.

Not fixed / needs follow-up in the KiCad GUI:
- 4 remaining shorts (Column 8 x2, Column 9 x1, plus S1/S2 stabilizer
  holes) where the second colliding item couldn't be identified headlessly
  (no via, no pad at the exact coordinate) - KiCad's DRC panel highlights
  these interactively, which this toolset can't replicate.
- ~35 clearance-only violations from tightly interleaved Column 6 /
  LED-DOUT autorouted traces elsewhere on the board - a separate root
  cause, left untouched to avoid introducing new shorts blind.

IMPORTANT: the KiCad MCP backend (SWIG/pcbnew Python subprocess) crashed
partway through this session and did not come back, so these two fixes
were completed via direct .kicad_pcb text edits and hand-verified
clearance math rather than a live re-run of DRC. Please re-run DRC in
KiCad before merging to confirm no regressions, and close any open KiCad
session on this board first (lock files indicate it was open during this
work).

Co-Authored-By: Claude Sonnet 5 <noreply@anthropic.com>
Routing:
- net Row 3: track 446.2 -> 448.6 mm
- net Row 2: track 443.5 -> 444.2 mm
Changed lines of the file:
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@@
 		(fp_line
 			(start 9.03125 8.000001)
-			(end 14.78125 8)
+			(end 14.78125 7.999999)
 			(stroke
 				(width 0.05)
@@
 			(start 15.28125 7.500002)
 			(mid 15.134803 7.853553)
-			(end 14.78125 8)
+			(end 14.78125 7.999999)
 			(stroke
 				(width 0.05)
@@
 	)
 	(segment
-		(start 392.871437 166.56119)
-		(end 392.871437 166.687223)
-		(width 0.2)
-		(layer "B.Cu")
-		(net "")
-	)
-	(segment
-		(start 392.871437 166.687223)
-		(end 392.861328 166.697332)
-		(width 0.2)
-		(layer "B.Cu")
-		(net "")
-	)
-	(segment
 		(start 293.691437 117.36119)
 		(end 294.006667 117.36119)
@@
 	)
 	(segment
-		(start 125.392687 185.17619)
-		(end 121.982687 188.58619)
-		(width 0.2)
-		(layer "B.Cu")
-		(net "Row 3")
-	)
-	(segment
-		(start 149.528937 185.17619)
-		(end 125.392687 185.17619)
-		(width 0.2)
-		(layer "B.Cu")
-		(net "Row 3")
-	)
-	(segment
 		(start 223.512569 187.5258)
 		(end 227.255538 183.782831)
@@
 	)
 	(segment
+		(start 149.528937 185.17619)
+		(end 127.5 185.17619)
+		(width 0.2)
+		(layer "B.Cu")
+		(net "Row 3")
+	)
+	(segment
+		(start 127.5 185.17619)
+		(end 127.5 189.0)
+		(width 0.2)
+		(layer "B.Cu")
+		(net "Row 3")
+	)
+	(segment
+		(start 127.5 189.0)
+		(end 121.982687 188.58619)
+		(width 0.2)
+		(layer "B.Cu")
+		(net "Row 3")
+	)
+	(segment
 		(start 165.555837 190.429441)
 		(end 154.782188 190.429441)
@@
 	(segment
 		(start 406.780187 152.86744)
+		(end 406.780187 161.5)
+		(width 0.2)
+		(layer "B.Cu")
+		(net "Row 2")
+	)
+	(segment
+		(start 406.780187 161.5)
+		(end 405.8 164.0)
+		(width 0.2)
+		(layer "B.Cu")
+		(net "Row 2")
+	)
+	(segment
+		(start 405.8 164.0)
+		(end 405.8 168.4)
+		(width 0.2)
+		(layer "B.Cu")
+		(net "Row 2")
+	)
+	(segment
+		(start 405.8 168.4)
+		(end 406.780187 168.9)
+		(width 0.2)
+		(layer "B.Cu")
+		(net "Row 2")
+	)
+	(segment
+		(start 406.780187 168.9)
 		(end 406.780187 169.53619)
 		(width 0.2)
